File: keyboard-pcb-tutorial.kicad_pcb (KiCad board)
At the start: 2 copper layers, 72.2 x 38.1 mm, 24 parts, among them SW1 SW_Push, U1 ATmega32U4-AU, Y1 16MHz

Commit message: Finished routing
Parts:
- moved C1 10.3 mm to (58.4, 30.5), turned to 90 degrees
- moved C2 10.0 mm to (49.5, 30.5), turned to 270 degrees
- moved R2 0.79 mm to (37.3, 35.2)
- moved USB1 0.30 mm to (36.1, 25.4)
- moved C6 0.16 mm to (58.1, 54.1)
- moved R3 0.16 mm to (34.1, 35.2)
- turned F1 to 90 degrees
- turned R1 to 90 degrees
- turned Y1 to 180 degrees
Connections:
- U1 pad 27: Net-(U1-Pad27) -> ROW0
- U1 pad 28: Net-(U1-Pad28) -> COL1
- U1 pad 29: Net-(U1-Pad29) -> COL0
- U1 pad 30: Net-(U1-Pad30) -> ROW1
Routing:
- net GND: track 0.00 -> 140.2 mm
- net +5V: track 0.00 -> 105.8 mm, vias 0 -> 5
- net COL1: track 0.00 -> 50.7 mm
- net ROW1: track 0.00 -> 49.8 mm
- net ROW0: track 0.00 -> 47.0 mm
- net COL0: track 0.00 -> 31.5 mm
- net Net-(R1-Pad1): track 0.00 -> 30.2 mm, vias 0 -> 2
- net Net-(R3-Pad1): track 0.00 -> 21.2 mm
- net Net-(R2-Pad1): track 0.00 -> 20.3 mm
- net Net-(C2-Pad1): track 0.00 -> 13.1 mm
- net Net-(C1-Pad1): track 0.00 -> 11.8 mm
- net VCC: track 0.00 -> 10.2 mm
- net Net-(D2-Pad2): track 0.00 -> 7.06 mm
- net Net-(D1-Pad2): track 0.00 -> 7.06 mm
- net Net-(D4-Pad2): track 0.00 -> 7.06 mm
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- added copper zone on B.Cu, net GND
Other:
- board size 72.2 x 38.1 mm -> 73.8 x 38.1 mm
- net class Default: trace_width 0.25 -> 0.254
- net class Power added: clearance 0.2, trace_width 0.381, via_dia 0.8, via_drill 0.4
- board text added: "4-Key Macro Tutorial"
